Commit message: :tada: add free joint link to the environment

File: gym_pybullet_drones/assets/cf2x.urdf (robot description, URDF)
Before this commit: robot cf2, 6 links, 5 joints
Links:
- added link rope_end, mass 0.0001; collision sphere radius=.01; visual sphere radius=.01
- added link virtual_link0, mass 0
Joints:
- added joint joint0_x: type revolute, parent center_of_mass_link, child virtual_link0, origin xyz=0 0 0.0 rpy=0 0 0, axis 1 0 0, limit lower=-10000 upper=10000 effort=1000.0 velocity=1000.0
- added joint joint0_y: type revolute, parent virtual_link0, child rope_end, origin xyz=0 0 0.0 rpy=0 0 0, axis 0 1 0, limit lower=-10000 upper=10000 effort=1000.0 velocity=1000.0
